File: PCB/_autosave-kaniharu.kicad_pcb (KiCad board)
At the start: 4 copper layers, 75.1 x 50.4 mm, 97 parts, among them J2 USB_C_Receptacle_USB2.0_14P, J3 Conn_02x03_Odd_Even, J4 Conn_02x03_Odd_Even, J5 Conn_02x03_Odd_Even, J6 RJ45_Pulse_JXD6-0001NL, U1 STM32H723VGTx, U2 ISO1044BD, U3 ISO1044BD, U4 AZ1117-3.3, U6 DP83848C, U7 ISO1044BD, Y1 CSTNE16M0V53C000R0, Y2 50M

Commit message: update
Parts:
- moved R11 85.8 mm to (130.8, 103.4), turned to 90 degrees
- moved R9 79.9 mm to (122.0, 101.5)
- moved JP3 76.5 mm to (133.1, 100.2)
- moved JP1 76.3 mm to (118.7, 98.0)
- moved R10 38.3 mm to (106.8, 142.5)
- moved JP2 38.3 mm to (112.1, 134.7)
- moved C8 2.21 mm to (132.6, 97.2)
- moved C10 1.39 mm to (133.4, 95.7)
Routing:
- net /CAN3/CAN3H: track 6.27 -> 13.2 mm
- net /CAN3/CAN3L: track 9.52 -> 15.5 mm
- net +3.3V: track 41.0 -> 36.4 mm
- net Net-(JP3-B): track 0.00 -> 2.91 mm
Changed lines of the file:
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@@
 	(footprint "Resistor_SMD:R_0402_1005Metric_Pad0.72x0.64mm_HandSolder"
 		(layer "F.Cu")
-		(at 89.0782 178.3744)
+		(at 130.7592 103.3913 90)
 		(descr "Resistor SMD 0402 (1005 Metric), square (rectangular) end terminal, IPC-7351 nominal with elongated pad for handsoldering. (Body size source: IPC-SM-782 page 72, https://www.pcb-3d.com/wordpress/wp-content/uploads/ipc-sm-782a_amendment_1_and_2.pdf), generated with kicad-footprint-generator")
 		(tags "resistor handsolder")
 		(property "Reference" "R11"
-			(at 0 -1.17 0)
+			(at 0 -1.17 90)
 			(layer "F.SilkS")
 			(effects
@@
 		)
 		(property "Value" "R"
-			(at 0 1.17 0)
+			(at 0 1.17 90)
 			(layer "F.Fab")
 			(effects
@@
 		)
 		(property "Datasheet" ""
-			(at 0 0 0)
+			(at 0 0 90)
 			(layer "F.Fab")
 			(hide yes)
@@
 		)
 		(property "Description" "Resistor"
-			(at 0 0 0)
+			(at 0 0 90)
 			(layer "F.Fab")
 			(hide yes)
@@
 		)
 		(fp_line
-			(start -1.11 -0.47)
-			(end 1.11 -0.47)
+			(start 1.11 -0.47)
+			(end 1.11 0.47)
 			(stroke
 				(width 0.05)
@@
 		)
 		(fp_line
-			(start -1.11 0.47)
-			(end -1.11 -0.47)
+			(start -1.11 -0.47)
+			(end 1.11 -0.47)
 			(stroke
 				(width 0.05)
@@
 		)
 		(fp_line
-			(start 1.11 -0.47)
-			(end 1.11 0.47)
+			(start 1.11 0.47)
+			(end -1.11 0.47)
 			(stroke
 				(width 0.05)
@@
 		)
 		(fp_line
-			(start 1.11 0.47)
-			(end -1.11 0.47)
+			(start -1.11 0.47)
+			(end -1.11 -0.47)
 			(stroke
 				(width 0.05)
@@
 		)
 		(fp_line
-			(start -0.525 -0.27)
-			(end 0.525 -0.27)
+			(start 0.525 -0.27)
+			(end 0.525 0.27)
 			(stroke
 				(width 0.1)
@@
 		)
 		(fp_line
-			(start -0.525 0.27)
-			(end -0.525 -0.27)
+			(start -0.525 -0.27)
+			(end 0.525 -0.27)
 			(stroke
 				(width 0.1)
@@
 		)
 		(fp_line
-			(start 0.525 -0.27)
-			(end 0.525 0.27)
+			(start 0.525 0.27)
+			(end -0.525 0.27)
 			(stroke
 				(width 0.1)
@@
 		)
 		(fp_line
-			(start 0.525 0.27)
-			(end -0.525 0.27)
+			(start -0.525 0.27)
+			(end -0.525 -0.27)
 			(stroke
 				(width 0.1)
@@
 		)
 		(fp_text user "${REFERENCE}"
-			(at 0 0 0)
+			(at 0 0 90)
 			(layer "F.Fab")
 			(effects
@@
 		)
 		(pad "1" smd roundrect
-			(at -0.5975 0)
+			(at -0.5975 0 90)
 			(size 0.715 0.64)
 			(layers "F.Cu" "F.Mask" "F.Paste")
@@
 		)
 		(pad "2" smd roundrect
-			(at 0.5975 0)
+			(at 0.5975 0 90)
 			(size 0.715 0.64)
 			(layers "F.Cu" "F.Mask" "F.Paste")
@@
 	(footprint "Capacitor_SMD:C_0402_1005Metric_Pad0.74x0.62mm_HandSolder"
 		(layer "F.Cu")
-		(at 133.2801 97.0644 180)
+		(at 133.3667 95.6818 180)
 		(descr "Capacitor SMD 0402 (1005 Metric), square (rectangular) end terminal, IPC-7351 nominal with elongated pad for handsoldering. (Body size source: IPC-SM-782 page 76, https://www.pcb-3d.com/wordpress/wp-content/uploads/ipc-sm-782a_amendment_1_and_2.pdf), generated with kicad-footprint-generator")
 		(tags "capacitor handsolder")
@@
 	(footprint "Connector_PinHeader_2.54mm:PinHeader_1x02_P2.54mm_Vertical"
 		(layer "F.Cu")
-		(at 89.7382 168.5544)
+		(at 118.6688 97.9628)
 		(descr "Through hole straight pin header, 1x02, 2.54mm pitch, single row")
 		(tags "Through hole pin header THT 1x02 2.54mm single row")
@@
 		(tags "capacitor handsolder")
 		(property "Reference" "C31"
-			(at 0.2627 -1.1684 0)
+			(at -0.0167 1.016 0)
 			(layer "F.SilkS")
 			(effects
@@
 	(footprint "Connector_PinHeader_2.54mm:PinHeader_1x02_P2.54mm_Vertical"
 		(layer "F.Cu")
-		(at 98.9182 168.5544)
+		(at 133.1468 100.1776)
 		(descr "Through hole straight pin header, 1x02, 2.54mm pitch, single row")
 		(tags "Through hole pin header THT 1x02 2.54mm single row")
 		(property "Reference" "JP3"
-			(at 0 -2.38 0)
+			(at 0 5.2578 0)
 			(layer "F.SilkS")
 			(effects
@@
 	(footprint "Capacitor_SMD:C_0805_2012Metric_Pad1.18x1.45mm_HandSolder"
 		(layer "F.Cu")
-		(at 134.0675 98.8678 180)
+		(at 132.588 97.2312 180)
 		(descr "Capacitor SMD 0805 (2012 Metric), square (rectangular) end terminal, IPC-7351 nominal with elongated pad for handsoldering. (Body size source: IPC-SM-782 page 76, https://www.pcb-3d.com/wordpress/wp-content/uploads/ipc-sm-782a_amendment_1_and_2.pdf, https://docs.google.com/spreadsheets/d/1BsfQQcO9C6DZCsRaXUlFlo91Tg2WpOkGARC1WS5S8t0/edit?usp=sharing), generated with kicad-footprint-generator")
 		(tags "capacitor handsolder")
 		(property "Reference" "C8"
-			(at 0 -1.68 0)
+			(at 1.3716 1.6002 0)
 			(layer "F.SilkS")
 			(effects
@@
 	(footprint "Connector_PinHeader_2.54mm:PinHeader_1x02_P2.54mm_Vertical"
 		(layer "F.Cu")
-		(at 94.3282 168.5544)
+		(at 112.0902 134.6708)
 		(descr "Through hole straight pin header, 1x02, 2.54mm pitch, single row")
 		(tags "Through hole pin header THT 1x02 2.54mm single row")
@@
 	(footprint "Resistor_SMD:R_0402_1005Metric_Pad0.72x0.64mm_HandSolder"
 		(layer "F.Cu")
-		(at 89.0782 174.3944)
+		(at 121.9708 101.5492)
 		(descr "Resistor SMD 0402 (1005 Metric), square (rectangular) end terminal, IPC-7351 nominal with elongated pad for handsoldering. (Body size source: IPC-SM-782 page 72, https://www.pcb-3d.com/wordpress/wp-content/uploads/ipc-sm-782a_amendment_1_and_2.pdf), generated with kicad-footprint-generator")
 		(tags "resistor handsolder")
@@
 	(footprint "Resistor_SMD:R_0402_1005Metric_Pad0.72x0.64mm_HandSolder"
 		(layer "F.Cu")
-		(at 89.0782 176.3844)
+		(at 106.8402 142.5008)
 		(descr "Resistor SMD 0402 (1005 Metric), square (rectangular) end terminal, IPC-7351 nominal with elongated pad for handsoldering. (Body size source: IPC-SM-782 page 72, https://www.pcb-3d.com/wordpress/wp-content/uploads/ipc-sm-782a_amendment_1_and_2.pdf), generated with kicad-footprint-generator")
 		(tags "resistor handsolder")
@@
 	)
 	(segment
-		(start 133.8476 97.5303)
-		(end 133.8476 97.0644)
-		(width 0.25)
-		(layer "F.Cu")
-		(net 2)
-	)
-	(segment
 		(start 151.8277 125.403)
 		(end 151.8412 125.4165)
@@
 	)
 	(segment
-		(start 134.258 97.9407)
-		(end 133.8476 97.5303)
-		(width 0.25)
-		(layer "F.Cu")
-		(net 2)
-	)
-	(segment
 		(start 153.5027 119.3604)
 		(end 155.3101 119.3604)
@@
 	)
 	(segment
-		(start 135.105 98.2035)
-		(end 134.8422 97.9407)
-		(width 0.25)
-		(layer "F.Cu")
-		(net 2)
-	)
-	(segment
 		(start 146.8096 92.6702)
 		(end 146.7588 92.6702)
@@
 	)
 	(segment
-		(start 134.8422 97.9407)
-		(end 134.258 97.9407)
-		(width 0.25)
-		(layer "F.Cu")
-		(net 2)
-	)
-	(segment
 		(start 155.3101 119.3604)
 		(end 155.6004 119.6507)
@@
 	)
 	(segment
-		(start 133.8476 97.0644)
-		(end 135.7656 97.0644)
-		(width 0.2)
-		(layer "F.Cu")
-		(net 2)
-	)
-	(segment
 		(start 146.6598 92.5712)
 		(end 144.0974 92.5712)
@@
 	)
 	(segment
-		(start 135.105 98.8678)
-		(end 135.105 98.2035)
-		(width 0.25)
-		(layer "F.Cu")
-		(net 2)
-	)
-	(segment
 		(start 151.3277 108.1854)
 		(end 151.3277 109.5447)
@@
 	)
 	(segment
+		(start 131.1656 100.1776)
+		(end 133.1468 100.1776)
+		(width 0.25)
+		(layer "F.Cu")
+		(net 51)
+	)
+	(segment
 		(start 123.7692 91.2447)
 		(end 124.9452 92.4207)
@@
 	)
 	(segment
+		(start 129.3876 98.3996)
+		(end 131.1656 100.1776)
+		(width 0.25)
+		(layer "F.Cu")
+		(net 51)
+	)
+	(segment
 		(start 124.9452 92.4207)
 		(end 124.9452 94.083816)
@@
 	)
 	(segment
+		(start 129.3876 96.9294)
+		(end 129.3876 98.3996)
+		(width 0.25)
+		(layer "F.Cu")
+		(net 51)
+	)
+	(segment
+		(start 128.1176 97.76741)
+		(end 130.7592 100.40901)
+		(width 0.25)
+		(layer "F.Cu")
+		(net 53)
+	)
+	(segment
 		(start 125.4506 95.5548)
 		(end 127.717999 95.5548)
@@
 	)
 	(segment
+		(start 130.7592 100.40901)
+		(end 130.7592 102.7938)
+		(width 0.25)
+		(layer "F.Cu")
+		(net 53)
+	)
+	(segment
 		(start 128.1176 95.954401)
 		(end 128.1176 96.9294)
@@
 	)
 	(segment
+		(start 128.1176 96.9294)
+		(end 128.1176 97.76741)
+		(width 0.25)
+		(layer "F.Cu")
+		(net 53)
+	)
+	(segment
 		(start 123.7692 93.7847)
 		(end 123.7692 93.8734)
@@
 	)
 	(segment
+		(start 130.7592 103.9888)
+		(end 131.8756 103.9888)
+		(width 0.2)
+		(layer "F.Cu")
+		(net 57)
+	)
+	(segment
+		(start 131.8756 103.9888)
+		(end 133.1468 102.7176)
+		(width 0.2)
+		(layer "F.Cu")
+		(net 57)
+	)
+	(segment
