File: PCB_v2/MCU.kicad_sch (KiCad schematic)
At the start: 9 parts, among them J1 Conn_01x04, SW1 SW_Push, U1 STM32G473RCTx, Y1 CSTNE16M0V53C000R0

Commit message: 動いたからコミット
Parts:
- added C24: 1u, Capacitor_SMD:C_0603_1608Metric, symbol Device:C
- added R43: 10k, Resistor_SMD:R_0402_1005Metric, symbol Device:R
- C15, C16, C17, C18, C19: footprint Capacitor_SMD:C_0603_1608Metric_Pad1.08x0.95mm_HandSolder -> Capacitor_SMD:C_0402_1005Metric
Connections:
- net +3.3V: now also R43.2
- net GND: now also SW1.1, C24.2
- net NRST: now also SW1.2, U1.7 (PG10), C24.1, R43.1
- net W5500_RST: now reaches U1.17 (PA3)
- net USART1_TX: now reaches U1.22 (PC4)
- net USART1_RX: now reaches U1.23 (PC5)
Other:
- moved on the sheet: SW1, Y1
