File: PCB_v2/PCB_v2.kicad_sch (KiCad schematic)
At the start: 11 parts, among them J3 Conn_02x03_Odd_Even, J4 Conn_02x03_Odd_Even, U4 AZ1117-3.3

Commit message: 動いたからコミット
Parts:
- removed J3, J4: Conn_02x03_Odd_Even, Connector_IDC:IDC-Header_2x03_P2.54mm_Horizontal, symbol Connector_Generic:Conn_02x03_Odd_Even
- removed JP1, JP2: Jumper_2_Open, Connector_PinHeader_2.54mm:PinHeader_1x02_P2.54mm_Vertical, symbol Jumper:Jumper_2_Open
- added C25: 10u, Capacitor_SMD:C_0805_2012Metric, symbol Device:C
- added C26: 1u, Capacitor_SMD:C_0603_1608Metric, symbol Device:C
- added C8, C9: 0.1u, Capacitor_SMD:C_0402_1005Metric, symbol Device:C
- added D1, D2: LED_ARGB, 0_mylib:XL-1608RGBC, symbol Device:LED_ARGB
- added D4: D, 0_syslib:SODFL3618X110N, symbol Device:D
- added H1, H2, H3: MountingHole_Pad, MountingHole:MountingHole_3.2mm_M3, symbol Mechanical:MountingHole_Pad
- added H4: MountingHole_Pad, MountingHole:MountingHole_3.2mm_M3_Pad, symbol Mechanical:MountingHole_Pad
- added J2, J3, J4: Conn_01x04, Connector_JST:JST_XA_S04B-XASK-1_1x04_P2.50mm_Horizontal, symbol Connector_Generic:Conn_01x04
- added L1: 22u, Inductor_SMD:L_0805_2012Metric_Pad1.15x1.40mm_HandSolder, symbol Device:L
- added PS1: RFM-0505S, 0_mylib:RFM-0505S, symbol 0_mylib:RFM-0505S
- added R11: 120, Resistor_SMD:R_0402_1005Metric, symbol Device:R
- added R37, R38, R39, R40, R41, R42: 1k, Resistor_SMD:R_0402_1005Metric, symbol Device:R
- C20, C21: footprint Capacitor_SMD:C_0805_2012Metric_Pad1.18x1.45mm_HandSolder -> Capacitor_SMD:C_0805_2012Metric
- R10, R9: value R -> 120; footprint Resistor_SMD:R_0603_1608Metric_Pad0.98x0.95mm_HandSolder -> Resistor_SMD:R_0402_1005Metric
- R36: footprint Resistor_SMD:R_0603_1608Metric_Pad0.98x0.95mm_HandSolder -> Resistor_SMD:R_0402_1005Metric
Connections:
- net +3.3V: now also C8.1, C9.1, D1.1 (A), D2.1 (A)
- net +5V: now also D4.1 (K)
- net +5VA: now also C25.1, J2.1 (Pin_1), J3.1 (Pin_1), J4.1 (Pin_1), L1.1
- net GND: now also C26.2, C8.2, C9.2, H4.1, PS1.3 (-VOUT)
- net GNDPWR: now also C25.2, J2.2 (Pin_2), J3.2 (Pin_2), J4.2 (Pin_2), PS1.1 (-VIN)
- net CAN1/CAN1L: now reaches R9.1
- net CAN1/CAN1L: now also J2.4 (Pin_4)
- net CAN1/CAN1H: now reaches R9.2
- net CAN1/CAN1H: now also J2.3 (Pin_3)
- net CAN3/CAN3L: now reaches R10.1
- net CAN3/CAN3L: now also J4.4 (Pin_4)
- net CAN3/CAN3H: now reaches R10.2
- net CAN3/CAN3H: now also J4.3 (Pin_3)
- new net: C26.1, D4.2 (A), PS1.4 (+VOUT)
- new net: D1.3 (GK), R37.1
- new net: L1.2, PS1.2 (+VIN)
- new net: D2.3 (GK), R40.1
- new net: D2.4 (BK), R39.1
- new net: D1.4 (BK), R42.1
- new net: D1.2 (RK), R38.1
- new net: D2.2 (RK), R41.1
- new net CAN2/CAN2H: J3.3 (Pin_3), R11.2
- new net CAN2/CAN2L: J3.4 (Pin_4), R11.1
- new net MCU/TIM1_CH1: R40.2
- new net MCU/TIM1_CH2: R39.2
- new net MCU/TIM1_CH3: R41.2
- new net MCU/TIM2_CH1: R37.2
- new net MCU/TIM2_CH2: R42.2
- new net MCU/TIM2_CH3: R38.2
- no-connect marks 4 -> 3
Other:
- added sheet CAN2 (CAN2.kicad_sch)
- added sheet CAN3 (CAN3.kicad_sch)
- added sheet SERIAL (SERIAL.kicad_sch)
- sheet CAN1 ports: added CAN1H, CAN1L, FDCAN1_RX, FDCAN1_TX; removed none
- sheet MCU ports: added FDCAN1_RX, FDCAN1_TX, FDCAN2_RX, FDCAN2_TX, FDCAN3_RX, FDCAN3_TX, SPI1_CS, SPI1_MISO, SPI1_MOSI, SPI1_SCK, TIM1_CH1, TIM1_CH2, TIM1_CH3, TIM2_CH1, TIM2_CH2, TIM2_CH3, USART1_RX, USART1_TX, W5500_RST; removed none
- moved on the sheet: R10, R9
